File: nepcropad.kicad_pcb (KiCad board)
At the start: 2 copper layers, 92.9 x 58.7 mm, 34 parts, among them SW1 SW_Push, U1 ATmega32U4-A, Y1 16MHz

Commit message: Done for the night
Parts:
- SW1: moved to B.Cu
- moved R3 8.78 mm to (88.9, 72.2), turned to -90 degrees
- moved R2 7.98 mm to (92.9, 72.2), turned to -90 degrees
- moved USB1 7.94 mm to (91.3, 62.7)
- moved F1 6.35 mm to (88.1, 77.0)
- moved C7 5.32 mm to (101.6, 98.4), turned to -90 degrees
- moved C3 1.59 mm to (101.6, 89.7)
- moved C4 0.79 mm to (103.2, 83.3)
- moved R1 0.79 mm to (100.0, 83.3), turned to -90 degrees
- turned SW1 to 180 degrees
Routing:
- net GND: track 0.00 -> 95.8 mm
- net Net-(R3-Pad2): track 0.00 -> 33.3 mm
- net Net-(R2-Pad2): track 0.00 -> 31.7 mm
- net +5V: track 0.00 -> 22.6 mm
- net Net-(R1-Pad2): track 0.00 -> 16.9 mm, vias 0 -> 2
- net Net-(C2-Pad2): track 0.00 -> 12.0 mm
- net Net-(C1-Pad2): track 0.00 -> 9.52 mm
- net VCC: track 0.00 -> 5.74 mm
- net D+: track 0.00 -> 4.77 mm
- net D-: track 0.00 -> 4.77 mm
- net Net-(C3-Pad1): track 0.00 -> 3.53 mm
Other:
- board size 92.9 x 58.7 mm -> 99.2 x 58.7 mm

Commit message: Finished routing of SoC area
Still need to finish routing of the keyswitch matrix.
I wired the switches together, but not to the soc
Parts:
- moved F1 3.97 mm to (84.9, 79.4)
Routing:
- net +5V: track 22.6 -> 119.6 mm, vias 0 -> 5
- net GND: track 95.8 -> 147.2 mm
- net ROW2: track 0.00 -> 39.3 mm
- net ROW1: track 0.00 -> 39.3 mm
- net ROW0: track 0.00 -> 39.2 mm
- net COL2: track 0.00 -> 38.1 mm
- net COL1: track 0.00 -> 38.1 mm
- net COL0: track 0.00 -> 38.1 mm
- net VCC: track 5.74 -> 16.4 mm
- net Net-(R1-Pad2): track 16.9 -> 27.2 mm
- net Net-(D2-Pad2): track 0.00 -> 7.77 mm
- net Net-(D9-Pad2): track 0.00 -> 7.71 mm
- net Net-(D7-Pad2): track 0.00 -> 7.71 mm
- net Net-(D6-Pad2): track 0.00 -> 7.71 mm
- net Net-(D4-Pad2): track 0.00 -> 7.71 mm
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